Commit message: Added RealSense Camera, Hsai Lidar, filenames modified to search the package
Signed-off-by: aaggj <albertogarciagomezjacinto@gmail.com>

File: go2_description/urdf/go2_description.urdf (robot description, URDF)
Before this commit: robot go2_description, 29 links, 28 joints
Links:
- added link camera_link; collision cylinder length=0.09 radius=0.05; visual cylinder length=0.01 radius=0.01
- added link camera_optical_link; collision cylinder length=0.09 radius=0.05; visual cylinder length=0.01 radius=0.01
- added link camera_support_link; collision cylinder length=0.09 radius=0.05; visual cylinder length=0.01 radius=0.01
- added link hesai_lidar; collision cylinder length=0.09 radius=0.05; visual cylinder length=0.09 radius=0.05
- added link odom
- link FL_calf: geometry collision cylinder length=0.12 radius=0.012; visual mesh filename=file://$(find go2_description)/dae/calf.dae
- link FL_foot: geometry collision sphere radius=0.022; visual mesh filename=file://$(find go2_description)/dae/foot.dae
- link FL_hip: geometry collision cylinder length=0.04 radius=0.046; visual mesh filename=file://$(find go2_description)/dae/hip.dae
- link FL_thigh: geometry collision box size=0.213 0.0245 0.034; visual mesh filename=file://$(find go2_description)/dae/thigh.dae
- link FR_calf: geometry collision cylinder length=0.12 radius=0.013; visual mesh filename=file://$(find go2_description)/dae/calf_mirror.dae
- link FR_foot: geometry collision sphere radius=0.022; visual mesh filename=file://$(find go2_description)/dae/foot.dae
- link FR_hip: geometry collision cylinder length=0.04 radius=0.046; visual mesh filename=file://$(find go2_description)/dae/hip.dae
- link FR_thigh: geometry collision box size=0.213 0.0245 0.034; visual mesh filename=file://$(find go2_description)/dae/thigh_mirror.dae
- link RL_calf: geometry collision cylinder length=0.12 radius=0.013; visual mesh filename=file://$(find go2_description)/dae/calf.dae
- link RL_foot: geometry collision sphere radius=0.022; visual mesh filename=file://$(find go2_description)/dae/foot.dae
- link RL_hip: geometry collision cylinder length=0.04 radius=0.046; visual mesh filename=file://$(find go2_description)/dae/hip.dae
- link RL_thigh: geometry collision box size=0.213 0.0245 0.034; visual mesh filename=file://$(find go2_description)/dae/thigh.dae
- link RR_calf: geometry collision cylinder length=0.12 radius=0.013; visual mesh filename=file://$(find go2_description)/dae/calf_mirror.dae
- link RR_foot: geometry collision sphere radius=0.022; visual mesh filename=file://$(find go2_description)/dae/foot.dae
- link RR_hip: geometry collision cylinder length=0.04 radius=0.046; visual mesh filename=file://$(find go2_description)/dae/hip.dae
- link RR_thigh: geometry collision box size=0.213 0.0245 0.034; visual mesh filename=file://$(find go2_description)/dae/thigh_mirror.dae
- link base_link: geometry collision box size=0.3762 0.0935 0.114; visual mesh filename=file://$(find go2_description)/dae/base.dae
Joints:
- added joint camera_link_joint: type fixed, parent camera_support_link, child camera_link, origin xyz=0.04 0 0.18 rpy=0 0 0, axis 0 0 0
- added joint camera_optical_link_joint: type fixed, parent camera_link, child camera_optical_link, origin xyz=0.012 0 0 rpy=-1.5708 0 -1.5708, axis 0 0 0
- added joint camera_support_link_joint: type fixed, parent base_link, child camera_support_link, origin xyz=0.29 0 0.04 rpy=0 0 0, axis 0 0 0
- added joint hesai_lidar_joint: type fixed, parent base_link, child hesai_lidar, origin xyz=0.15 0 0.08 rpy=0 0 1.5708, axis 0 0 0
- added joint odom_joint: type fixed, parent odom, child base_link, origin xyz=0 0 0 rpy=0 0 0

Commit message: Camera and lidar calibration with point cloud and camera
Signed-off-by: aaggj <albertogarciagomezjacinto@gmail.com>

File: go2_description/urdf/go2_description.urdf (robot description, URDF)
Before this commit: robot go2_description, 34 links, 33 joints
Joints:
- joint camera_link_joint: origin xyz=0.04 0 0.18 rpy=0 0 0 -> xyz=0.04 0.03 0.018 rpy=0 -0.04 0
- joint camera_support_link_joint: origin xyz=0.29 0 0.04 rpy=0 0 0 -> xyz=0.29 0 0.0958 rpy=0 0 0
- joint hesai_lidar_joint: origin xyz=0.15 0 0.08 rpy=0 0 1.5708 -> xyz=0.15 0 0.12 rpy=0 0 1.5708
